File: INSUMOS/tralala-8088-homebrew-code-r196-trunk-hw-8088/pic_and_io.kicad_sch (KiCad schematic)
At the start: 0 parts

Commit message: Inicio da bios apos testes
Parts:
- added C18, C19: 22pF, Capacitor_THT:C_Disc_D6.0mm_W2.5mm_P5.00mm, symbol Device:C
- added C20, C21, C23: 100nF, Capacitor_THT:C_Disc_D6.0mm_W2.5mm_P5.00mm, symbol Device:C
- added C22: 220nF, Capacitor_THT:C_Disc_D6.0mm_W2.5mm_P5.00mm, symbol Device:C
- added D10, D9: 1N4148, Diode_THT:D_DO-35_SOD27_P7.62mm_Horizontal, symbol Diode:1N4148
- added D6: LED_RED, LED_THT:LED_D5.0mm, symbol Device:LED
- added D7: LED_YELLOW, LED_THT:LED_D5.0mm, symbol Device:LED
- added D8: LED_GREEN, LED_THT:LED_D5.0mm, symbol Device:LED
- added P5: Conn_01x02_Male, Connector_PinHeader_2.54mm:PinHeader_1x02_P2.54mm_Vertical, symbol Connector:Conn_01x02_Male
- added P6, P9: CONN_01X10, Connector_PinSocket_2.54mm:PinSocket_1x10_P2.54mm_Vertical, symbol Connector_Generic:Conn_01x10
- added P7: PIC ISP, Connector_IDC:IDC-Header_2x03_P2.54mm_Vertical, symbol Connector_Generic:Conn_02x03_Odd_Even
- added P8: USB_B, Connector_USB:USB_B_Lumberg_2411_02_Horizontal, symbol Connector_modified:USB_B
- added Q1, Q2, Q3: 2N3904, Package_TO_SOT_THT:TO-92_HandSolder, symbol Device:Q_NPN_EBC
- added R10, R11, R9: 100, Resistor_THT:R_Axial_DIN0207_L6.3mm_D2.5mm_P10.16mm_Horizontal, symbol Device:R
- added R12: 47K, Resistor_THT:R_Axial_DIN0207_L6.3mm_D2.5mm_P10.16mm_Horizontal, symbol Device:R
- added R6, R7, R8: 10K, Resistor_THT:R_Axial_DIN0207_L6.3mm_D2.5mm_P10.16mm_Horizontal, symbol Device:R
- added SW2: RESET_PIC, Button_Switch_THT:SW_PUSH_6mm_H5mm, symbol Switch:SW_Push
- added U15: PIC18(L)F4550-I/P or PIC18(L)F4553-I/P, Package_DIP:DIP-40_W15.24mm, symbol MCU_Microchip_PIC18:PIC18F4553-IP
- added Y2: 20.000 MHz, Crystal:Crystal_HC49-U_Vertical, symbol Device:Crystal
Connections:
- new net: C22.1, U15.18 (VUSB)
- new net: D10.1 (K), D9.1 (K), P5.1 (Pin_1), SW2.1, U15.1 (Vpp/~{MCLR}/RE3)
- new net: Q2.2 (B), R7.1
- new net: Q3.2 (B), R8.1
- new net: C19.2, U15.13 (OSC1/CLKI), Y2.2
- new net: Q3.3 (C), R11.2
- new net: C18.2, U15.14 (RA6/OSC2/CLKO), Y2.1
- new net: C23.1, D9.2 (A), R12.2
- new net: D7.1 (K), R10.1
- new net: Q2.3 (C), R10.2
- new net: P8.2 (D-), U15.23 (VM/D-/RC4)
- new net: P8.3 (D+), U15.24 (VP/D+/RC5)
- new net: Q1.2 (B), R6.1
- new net: Q1.3 (C), R9.2
- new net: D6.1 (K), R9.1
- new net: D8.1 (K), R11.1
- new net +5V: C20.1, C21.1, D6.2 (A), D7.2 (A), D8.2 (A), P7.2 (Pin_2), P9.1 (Pin_1), R12.1, U15.11 (VDD), U15.32 (VDD)
- new net GND: C18.1, C19.1, C20.2, C21.2, C22.2, C23.2, P5.2 (Pin_2), P7.5 (Pin_5), P7.6 (Pin_6), P8.4 (GND), P8.5 (Shield), P9.10 (Pin_10), Q1.1 (E), Q2.1 (E), Q3.1 (E), SW2.2, U15.12 (VSS), U15.31 (VSS)
- new net ICH_ACK: U15.36 (RB3/AN9/CCP2/VPO)
- new net ICH_D0: U15.19 (SPP0/RD0)
- new net ICH_D1: U15.20 (SPP1/RD1)
- new net ICH_D2: U15.21 (SPP2/RD2)
- new net ICH_D3: U15.22 (SPP3/RD3)
- new net ICH_D4: U15.27 (SPP4/RD4)
- new net ICH_D5: U15.28 (P1B/SPP5/RD5)
- new net ICH_D6: U15.29 (P1C/SPP6/RD6)
- new net ICH_D7: U15.30 (P1D/SPP7/RD7)
- new net ICH_IBF: U15.37 (RB4/AN11/KBI0/CSSPP)
- new net ICH_OBF: U15.35 (RB2/AN8/INT2/VMO)
- new net ICH_STB: U15.38 (RB5/KBI1/PGM)
- new net LED_GREEN: R8.2
- new net LED_RED: R6.2
- new net LED_YELLOW: R7.2
- new net PIC_PGC: P7.3 (Pin_3), U15.39 (RB6/KBI2/PGC)
- new net PIC_PGD: P7.4 (Pin_4), U15.40 (RB7/KBI3/PGD)
- new net PIC_VPP: D10.2 (A), P7.1 (Pin_1)
- new net TFT_D_C: P9.7 (Pin_7), U15.10 (OESPP/AN7/RE2)
- new net TFT_LCD_CS: P9.5 (Pin_5), U15.8 (CK1SPP/AN5/RE0)
- new net TFT_MISO: P9.2 (Pin_2), U15.33 (RB0/AN12/INT0/FLT0/SDI/SDA)
- new net TFT_MOSI: P9.4 (Pin_4), U15.26 (SDO/RX/DT/RC7)
- new net TFT_Reset: P9.8 (Pin_8), U15.25 (TX/CK/RC6)
- new net TFT_SCK: P9.3 (Pin_3), U15.34 (RB1/AN10/INT1/SCK/SCL)
- new net TFT_SD_CS: P9.6 (Pin_6), U15.9 (CK2SPP/AN6/RE1)
- no-connect marks 0 -> 21
