File: schematics/my_pcxt/8088system.kicad_sch (KiCad schematic)
At the start: 24 parts, among them J1 Conn_02x40_Top_Bottom, P11 ~{TEST}, P2 NMI, P4 Conn_01x02_Male, SW2 RESET_8088, U10 74HCT373, U11 8284, U12 74LS74, U13 74LS138, U4 8288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

Commit message: Implemented 8259 e 8253
Parts:
- removed J1: Conn_02x40_Top_Bottom, symbol Connector_Generic:Conn_02x40_Top_Bottom
- added J2: Conn_02x40_Top_Bottom, symbol Connector_Generic:Conn_02x40_Top_Bottom
- added unit 3 of U7
Connections:
- net +12V: now also J2.23 (Pin_23)
- net +5V: now also J2.18 (Pin_18), J2.29 (Pin_29), J2.3 (Pin_3), J2.58 (Pin_58)
- net -12V: now also J2.25 (Pin_25)
- net -5V: now also J2.27 (Pin_27)
- net 8259A_SP_EN: now also J2.78 (Pin_78)
- net AEN: now also J2.72 (Pin_72)
- net ALE: now also J2.4 (Pin_4)
- net BUF_A0: now also J2.41 (Pin_41)
- net BUF_A1: now also J2.42 (Pin_42)
- net BUF_A10: now also J2.51 (Pin_51)
- net BUF_A11: now also J2.52 (Pin_52)
- net BUF_A12: now also J2.53 (Pin_53)
- net BUF_A13: now also J2.54 (Pin_54)
- net BUF_A14: now also J2.55 (Pin_55)
- net BUF_A15: now also J2.56 (Pin_56)
- net BUF_A16: now also J2.59 (Pin_59)
- net BUF_A17: now also J2.60 (Pin_60)
- net BUF_A18: now also J2.61 (Pin_61)
- net BUF_A19: now also J2.62 (Pin_62)
- net BUF_A2: now also J2.43 (Pin_43)
- net BUF_A3: now also J2.44 (Pin_44)
- net BUF_A4: now also J2.45 (Pin_45)
- net BUF_A5: now also J2.46 (Pin_46)
- net BUF_A6: now also J2.47 (Pin_47)
- net BUF_A7: now also J2.48 (Pin_48)
- net BUF_A8: now also J2.49 (Pin_49)
- net BUF_A9: now also J2.50 (Pin_50)
- net BUF_D0: now also J2.63 (Pin_63)
- net BUF_D1: now also J2.64 (Pin_64)
- net BUF_D2: now also J2.65 (Pin_65)
- net BUF_D3: now also J2.66 (Pin_66)
- net BUF_D4: now also J2.67 (Pin_67)
- net BUF_D5: now also J2.68 (Pin_68)
- net BUF_D6: now also J2.69 (Pin_69)
- net BUF_D7: now also J2.70 (Pin_70)
- net CH_CK: now also J2.71 (Pin_71)
- net CLK88: now also J2.12 (Pin_12)
- net DACK1: now also J2.15 (Pin_15)
- net DACK2: now also J2.6 (Pin_6)
- net DRQ1: now also J2.14 (Pin_14)
- net DRQ2: now also J2.26 (Pin_26)
- net DRQ3: now also J2.16 (Pin_16)
- net GNDREF: now also J2.1 (Pin_1), J2.17 (Pin_17), J2.22 (Pin_22), J2.31 (Pin_31), J2.57 (Pin_57)
- net INTA: now also J2.39 (Pin_39)
- net INTR: now also J2.79 (Pin_79)
- net IORD: now also J2.24 (Pin_24)
- net IOWR: now also J2.19 (Pin_19)
- net IRQ2: now also J2.28 (Pin_28)
- net IRQ3: now also J2.7 (Pin_7)
- net IRQ4: now also J2.8 (Pin_8)
- net IRQ5: now also J2.9 (Pin_9)
- net IRQ6: now also J2.10 (Pin_10)
- net IRQ7: now also J2.11 (Pin_11)
- net MRD: now also J2.20 (Pin_20)
- net MWR: now also J2.21 (Pin_21)
- net OSC88: now also J2.2 (Pin_2)
- net RDY1: now also J2.73 (Pin_73)
- net RESOUT: now also J2.30 (Pin_30)
- net TC: now also J2.5 (Pin_5)
- net at U13.15 (O0): now also U7.10, U7.9; no longer U12.3 (C)
- net PCLK: now reaches U11.2 (PCLK)
- net PCLK: now also J2.77 (Pin_77)
- new net: U12.3 (C), U7.8
Other:
- moved on the sheet: U13

Commit message: Updating schematic
Parts:
- added C22: 10nF, symbol Device:C
- added J6: Conn_01x04, symbol Connector_Generic:Conn_01x04
- added LS1: Speaker, symbol Device:Speaker
- added Q1: 2N2219, Package_TO_SOT_THT:TO-39-3, symbol Transistor_BJT:2N2219
- added R3: 1K, Resistor_THT:R_Axial_DIN0207_L6.3mm_D2.5mm_P10.16mm_Horizontal, symbol Device:R
- added R4: 33R, Resistor_THT:R_Axial_DIN0207_L6.3mm_D2.5mm_P10.16mm_Horizontal, symbol Device:R
- added U24: 74LS00, symbol 74xx:74LS00
Connections:
- net +5V: now also J6.4 (Pin_4), LS1.2
- net GNDREF: now also C22.2, Q1.1 (E)
- net SPKR: now reaches J2.38 (Pin_38)
- net SPKR: now also U24.4, U24.5
- new net: J6.1 (Pin_1), R4.2
- new net: J6.2 (Pin_2), LS1.1
- new net: Q1.2 (B), R3.2
- new net: C22.1, Q1.3 (C), R4.1
- new net: R3.1, U24.6
- no-connect marks 22 -> 23

Commit message: Updating code...
Parts:
- removed C22: 10nF, symbol Device:C
- removed J6: Conn_01x04, symbol Connector_Generic:Conn_01x04
- removed LS1: Speaker, symbol Device:Speaker
- removed Q1: 2N2219, Package_TO_SOT_THT:TO-39-3, symbol Transistor_BJT:2N2219
- removed R3: 1K, Resistor_THT:R_Axial_DIN0207_L6.3mm_D2.5mm_P10.16mm_Horizontal, symbol Device:R
- removed R4: 33R, Resistor_THT:R_Axial_DIN0207_L6.3mm_D2.5mm_P10.16mm_Horizontal, symbol Device:R
- removed U24: 74LS00, symbol 74xx:74LS00
Connections:
- net BUF_D0: no longer U6.18 (B0)
- net BUF_D1: no longer U6.17 (B1)
- net BUF_D2: no longer U6.16 (B2)
- net BUF_D3: no longer U6.15 (B3)
- net BUF_D4: no longer U6.14 (B4)
- net BUF_D5: no longer U6.13 (B5)
- net BUF_D6: no longer U6.12 (B6)
- net BUF_D7: no longer U6.11 (B7)
- new net D0: U6.18 (B0)
- new net D1: U6.17 (B1)
- new net D2: U6.16 (B2)
- new net D3: U6.15 (B3)
- new net D4: U6.14 (B4)
- new net D5: U6.13 (B5)
- new net D6: U6.12 (B6)
- new net D7: U6.11 (B7)
- no-connect marks 23 -> 22
Other:
- moved on the sheet: U6
