File: schematics/my_pcxt/pic_timer_rs232.kicad_sch (KiCad schematic)
At the start: 17 parts, among them J3 Conn_02x40_Top_Bottom, J5 DE9_Plug, U14 16550, U15 8253, U23 DTE, U3 PAL20L8, U7 8259A, X1 4.915200MHz

Commit message: Updating schematic
Connections:
- net +5V: now also U14.12 (CS0), U14.13 (CS1); no longer U14.25 (~{ADS})
- net A3: no longer U14.12 (CS0)
- net A4: no longer U14.13 (CS1)
- net GNDREF: now also U14.25 (~{ADS}); no longer U14.36 (~{CTS})
Other:
- moved on the sheet: C12, C19, C20, C21, C2VS+1, C2VS-1, J5, U14, U23, X1

Commit message: Updating code...
Parts:
- added U25: 74LS08, symbol 74xx:74LS08
Connections:
- net AD0 is gone; now on net D0: U15.8 (D0), U7.11 (D0)
- net AD1 is gone; now on net D1: U15.7 (D1), U7.10 (D1)
- net AD2 is gone; now on net D2: U15.6 (D2), U7.9 (D2)
- net AD3 is gone; now on net D3: U15.5 (D3), U7.8 (D3)
- net AD4 is gone; now on net D4: U15.4 (D4), U7.7 (D4)
- net AD5 is gone; now on net D5: U15.3 (D5), U7.6 (D5)
- net AD6 is gone; now on net D6: U15.2 (D6), U7.5 (D6)
- net AD7 is gone; now on net D7: U15.1 (D7), U7.4 (D7)
- net +5V: now also U15.13 (OUT1); no longer U15.14 (G1), U15.16 (G2)
- net SPEAKER_DATA: now reaches U15.17 (OUT2)
- new net timer2GateSpeaker: U15.16 (G2)
