File: schematics/my_pcxt/pic_timer_rs232.kicad_sch (KiCad schematic)
At the start: 19 parts, among them J3 Conn_02x40_Top_Bottom, J5 DE9_Plug, P1 CH376S_0xE0, U14 16550, U15 8253, U23 DTE, U25 74LS08, U3 PAL20L8, U7 8259A, X1 4.915200MHz

Commit message: Updating...
Parts:
- added C22, C25, C26, C2VS+2, C2VS-2: 1uF, symbol Device:C_Polarized
- added U24: DTE, symbol Interface_UART:MAX232
Connections:
- net +5V: now also C25.1, C2VS+2.2, U24.16 (VCC); no longer U14.39 (~{RI})
- net GNDREF: now also J5.5, C25.2, C2VS-2.1; no longer U14.37 (~{DSR}), U14.38 (~{DCD})
- net /RTS: now reaches U14.32 (~{RTS})
- net /RTS: now also U23.11 (T1IN)
- net /DTR: now reaches U14.33 (~{DTR})
- net /DTR: now also U24.11 (T1IN)
- net /CTS: now reaches U14.36 (~{CTS})
- net /CTS: now also U23.12 (R1OUT)
- net CTS: now reaches U23.13 (R1IN)
- net CTS: now also J5.8
- net RTS: now reaches U23.14 (T1OUT)
- net RTS: now also J5.7
- net TX: now reaches J5.3, U23.7 (T2OUT)
- net RX: now reaches J5.2, U23.8 (R2IN)
- net DCD: now reaches J5.1
- net DCD: now also U24.7 (T2OUT)
- net DTR: now reaches J5.4
- net DTR: now also U24.14 (T1OUT)
- net DSR: now reaches J5.6
- net DSR: now also U24.13 (R1IN)
- net RI: now reaches J5.9
- net RI: now also U24.8 (R2IN)
- new net: C22.1, U24.1 (C1+)
- new net: C2VS+2.1, U24.2 (VS+)
- new net: C22.2, U24.3 (C1-)
- new net: C26.1, U24.4 (C2+)
- new net: C26.2, U24.5 (C2-)
- new net: C2VS-2.2, U24.6 (VS-)
- new net /DCD: U14.38 (~{DCD}), U24.10 (T2IN)
- new net /DSR: U14.37 (~{DSR}), U24.12 (R1OUT)
- new net /RI: U14.39 (~{RI}), U24.9 (R2OUT)
- no-connect marks 18 -> 12
