File: schematics/my_pcxt/my_pcxt.kicad_sch (KiCad schematic)
At the start: 5 parts, among them U1 74HCT00

Commit message: Updating schematics
Other:
- sheet pic_timer renamed pic_timer_rs232
- sheet pic_timer_rs232: file pic_timer.kicad_sch -> pic_timer_rs232.kicad_sch
Changed lines of the file:
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@@
     (stroke (width 0.1524) (type solid))
     (fill (color 0 0 0 0.0000))
-    (property "Sheetname" "pic_timer" (at 186.69 50.0884 0)
+    (property "Sheetname" "pic_timer_rs232" (at 186.69 50.0884 0)
       (effects (font (size 1.27 1.27)) (justify left bottom))
     )
-    (property "Sheetfile" "pic_timer.kicad_sch" (at 186.69 80.5946 0)
+    (property "Sheetfile" "pic_timer_rs232.kicad_sch" (at 186.69 80.5946 0)
       (effects (font (size 1.27 1.27)) (justify left top))
     )

Commit message: Implemented ch376s
Other:
- added sheet CH376S (CH376S.kicad_sch)
Changed lines of the file:
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@@
     )
   )
-  (sheet (at 127 25.4) (size 38.1 13.97) (fields_autoplaced)
+  (sheet (at 106.68 25.4) (size 25.4 12.7) (fields_autoplaced)
     (stroke (width 0.1524) (type solid))
     (fill (color 0 0 0 0.0000))
-    (property "Sheetname" "IO_8255" (at 127 24.6884 0)
+    (property "Sheetname" "IO_8255" (at 106.68 24.6884 0)
       (effects (font (size 1.27 1.27)) (justify left bottom))
     )
-    (property "Sheetfile" "IO_8255.kicad_sch" (at 127 39.9546 0)
+    (property "Sheetfile" "IO_8255.kicad_sch" (at 106.68 38.6846 0)
       (effects (font (size 1.27 1.27)) (justify left top))
     )
@@
     )
   )
-  (sheet (at 186.69 50.8) (size 41.91 29.21) (fields_autoplaced)
+  (sheet (at 134.62 25.4) (size 24.13 12.7) (fields_autoplaced)
     (stroke (width 0.1524) (type solid))
     (fill (color 0 0 0 0.0000))
-    (property "Sheetname" "pic_timer_rs232" (at 186.69 50.0884 0)
+    (property "Sheetname" "pic_timer_rs232" (at 134.62 24.6884 0)
       (effects (font (size 1.27 1.27)) (justify left bottom))
     )
-    (property "Sheetfile" "pic_timer_rs232.kicad_sch" (at 186.69 80.5946 0)
+    (property "Sheetfile" "pic_timer_rs232.kicad_sch" (at 134.62 38.6846 0)
       (effects (font (size 1.27 1.27)) (justify left top))
     )
@@
       )
     )
+  )
+  (sheet (at 165.1 25.4) (size 21.59 12.7) (fields_autoplaced)
+    (stroke (width 0.1524) (type solid))
+    (fill (color 0 0 0 0.0000))
+    (property "Sheetname" "CH376S" (at 165.1 24.6884 0)
+      (effects (font (size 1.27 1.27)) (justify left bottom))
+    )
+    (property "Sheetfile" "CH376S.kicad_sch" (at 165.1 38.6846 0)
+      (effects (font (size 1.27 1.27)) (justify left top))
+    )
+    (instances
+      (project "my_pcxt"
+        (path "/da0b7221-7a68-40fb-a49c-b89470148422" (page "7"))
+      )
+    )
